File: osmo-lea6t-gps/eagle/ublox-lea6-test.brd (EAGLE design)
At the start: 49.5 x 49.5 mm, 52 parts, among them U1 UBLOX-LEA-6T, U2 TPS73633, U3 TPS73633, X1 SERIAL, X2 ANT, X3 FOUT, X4 ANT, X5 FOUT, X6 1PPS, X7 PC, X8 1PPS, X9 22-23-2021

Commit message: mark R1 as 'DNP' (no stub to U.FL connector)
Parts:
- R1: value 0R -> DNP
Changed lines of the file:
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@@
 <attribute name="VALUE" x="4.6675" y="43.7275" size="1.27" layer="27" rot="R270"/>
 </element>
-<element name="R1" library="we_passive" package="0603" value="0R" x="5.715" y="41.275" smashed="yes">
+<element name="R1" library="we_passive" package="0603" value="DNP" x="5.715" y="41.275" smashed="yes">
 <attribute name="NAME" x="4.1275" y="39.0525" size="1.27" layer="25"/>
 <attribute name="VALUE" x="4.215" y="39.275" size="1.27" layer="27"/>
