File: osmo-lea6t-gps/eagle/ublox-lea6-test.sch (EAGLE design)
At the start: 52 parts, among them U1 UBLOX-LEA-6T, U2 TPS73633, U3 TPS73633, X1 SERIAL, X2 ANT, X3 FOUT, X4 ANT, X5 FOUT, X6 1PPS, X7 PC, X8 1PPS, X9 22-23-2021

Commit message: mark R1 as 'DNP' (no stub to U.FL connector)
Parts:
- R1: value 0R -> DNP
Changed lines of the file:
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@@
 <part name="TP7" library="we_conn" deviceset="TESTPAD" device=""/>
 <part name="R2" library="we_passive" deviceset="R-EU" device="_0603" value="0R"/>
-<part name="R1" library="we_passive" deviceset="R-EU" device="_0603" value="0R"/>
+<part name="R1" library="we_passive" deviceset="R-EU" device="_0603" value="DNP"/>
 <part name="X1" library="laforge" deviceset="JACK2.5_SJ-2523" device="" value="SERIAL"/>
 <part name="U$10" library="we_supply" deviceset="GND" device=""/>
