File: e1-tap/e1_tap.sch (EAGLE design)
At the start: 8 parts, among them J1 PASSTHROUGH, J2 TAP, SW1 CROSSOVER, SW2 TERM

Commit message: e1-tap: Add BOM attributes
Parts:
- J1, J2: CLASS (none) -> CONNECTOR\JUMPER; DESCRIPTION (none) -> CONN MOD JACK 8P8C R/A UNSHLD; LINK (none) -> https://www.digikey.de/product-detail/en/te-connectivity-am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; MANUFACTURER (none) -> TE Connectivity AMP Connectors; MANUFACTURERPARTNUMBER (none) -> 5557560-1; POPULATED (none) -> TRUE; ROHSCERTIFICATE (none) -> UNKNOWN ROHS CERTIFICATE; SOURCE (none) -> DIGIKEY; SOURCEPARTNUMBER (none) -> A31449-ND
- R1, R2, R3, R4: CLASS (none) -> RESISTOR; DESCRIPTION (none) -> RES SMD 1K OHM 1% 1/10W 0603; LINK (none) -> https://www.digikey.de/product-detail/en/yageo/RC0603FR-071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; MANUFACTURER (none) -> Yageo; MANUFACTURERPARTNUMBER (none) -> RC0603FR-071KL; POPULATED (none) -> TRUE; ROHSCERTIFICATE (none) -> UNKNOWN ROHS CERTIFICATE; SOURCE (none) -> DIGIKEY; SOURCEPARTNUMBER (none) -> 311-1.00KHRCT-ND
- SW1, SW2: CLASS (none) -> UNKNOWN CLASS; DESCRIPTION (none) -> SWITCH SLIDE 4PDT 300MA 115V; LINK (none) -> https://www.digikey.de/product-detail/en/te-connectivity-al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; MANUFACTURER (none) -> TE Connectivity ALCOSWITCH Switches; MANUFACTURERPARTNUMBER (none) -> 1-1825010-3; POPULATED (none) -> TRUE; ROHSCERTIFICATE (none) -> UNKNOWN ROHS CERTIFICATE; SOURCE (none) -> DIGIKEY; SOURCEPARTNUMBER (none) -> 450-1633-ND
