File: clock-converter/clock-converter.sch (EAGLE design)
At the start: 51 parts, among them K1 DC IN, M1 MENTOR_12701001, U1 LTC6957-4, U2 ADP151AUJZ, X1 IN+, X2 IN-, X3 OUT1, X4 OUT2, X5 IN+, X6 IN-, X7 OUT1, X8 OUT2

Commit message: clock-converter: Add attributes with digikey links
Parts:
- C1, C2, C6, C7: CLASS (none) -> CAPACITOR; DESCRIPTION (none) -> CAP CER 0.1UF 16V X7R 0603; LINK (none) -> https://www.digikey.de/product-detail/de/samsung-electro-me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; MANUFACTURER (none) -> Samsung Electro-Mechanics; MANUFACTURERPARTNUMBER (none) -> CL10B104KO8NNNC; POPULATED (none) -> TRUE; ROHSCERTIFICATE (none) -> Bleifrei / RoHS-konform; SOURCE (none) -> DIGIKEY; SOURCEPARTNUMBER (none) -> 1276-1005-1-ND
- C10, C8: CLASS (none) -> CAPACITOR; DESCRIPTION (none) -> CAP CER 4.7UF 16V X5R 0805; LINK (none) -> https://www.digikey.de/product-detail/de/samsung-electro-me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; MANUFACTURER (none) -> Samsung Electro-Mechanics; MANUFACTURERPARTNUMBER (none) -> CL21A475KOFNNNE; POPULATED (none) -> TRUE; ROHSCERTIFICATE (none) -> Bleifrei / RoHS-konform; SOURCE (none) -> DIGIKEY; SOURCEPARTNUMBER (none) -> 1276-1065-1-ND
- C11, C3, C4, C5, C9: CLASS (none) -> CAPACITOR; DESCRIPTION (none) -> CAP CER 10000PF 50V X7R 0603; LINK (none) -> https://www.digikey.de/product-detail/de/kemet/C0603C103M5R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; MANUFACTURER (none) -> KEMET; MANUFACTURERPARTNUMBER (none) -> C0603C103M5RACTU; POPULATED (none) -> TRUE; ROHSCERTIFICATE (none) -> Bleifrei / RoHS-konform; SOURCE (none) -> DIGIKEY; SOURCEPARTNUMBER (none) -> 399-7842-1-ND
- D1, D2, D3, D4: CLASS (none) -> DIODE; DESCRIPTION (none) -> SUPPRESSOR ESD 30VDC 0603 SMD; LINK (none) -> https://www.digikey.de/product-detail/de/eaton-electronics-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; MANUFACTURER (none) -> Eaton - Electronics Division; MANUFACTURERPARTNUMBER (none) -> 0603ESDA2-TR2; POPULATED (none) -> TRUE; ROHSCERTIFICATE (none) -> Bleifrei / RoHS-konform; SOURCE (none) -> DIGIKEY; SOURCEPARTNUMBER (none) -> 283-4156-1-ND
- D5: CLASS (none) -> DIODE; DESCRIPTION (none) -> DIODE ZENER 5.6V 3W DO214AC; LINK (none) -> https://www.digikey.de/product-detail/de/micro-commercial-c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; MANUFACTURER (none) -> Micro Commercial Co; MANUFACTURERPARTNUMBER (none) -> 3SMAJ5919B-TP; POPULATED (none) -> TRUE; ROHSCERTIFICATE (none) -> Bleifrei / RoHS-konform; SOURCE (none) -> DIGIKEY; SOURCEPARTNUMBER (none) -> 3SMAJ5919B-TPMSCT-ND
- D6: CLASS (none) -> DIODE; DESCRIPTION (none) -> DIODE SCHOTTKY 30V 800MA USC; LINK (none) -> https://www.digikey.de/product-detail/de/toshiba-semiconduc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; MANUFACTURER (none) -> Toshiba Semiconductor and Storage; MANUFACTURERPARTNUMBER (none) -> CUS08F30,H3F; POPULATED (none) -> TRUE; ROHSCERTIFICATE (none) -> Bleifrei / RoHS-konform; SOURCE (none) -> DIGIKEY; SOURCEPARTNUMBER (none) -> CUS08F30H3FCT-ND
- F1: CLASS (none) -> UNKNOWN CLASS; DESCRIPTION (none) -> PTC RESET FUSE 30V 200MA 1206; LINK (none) -> https://www.digikey.de/product-detail/de/0ZCJ0020FF2E/507-1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; MANUFACTURER (none) -> Bel Fuse Inc.; MANUFACTURERPARTNUMBER (none) -> 0ZCJ0020FF2E; POPULATED (none) -> TRUE; ROHSCERTIFICATE (none) -> Bleifrei / RoHS-konform; SOURCE (none) -> DIGIKEY; SOURCEPARTNUMBER (none) -> 507-1797-1-ND
- JP1, JP2, JP3, JP4: CLASS (none) -> CONNECTOR\JUMPER; DESCRIPTION (none) -> CONN HEADER VERT 3POS 2.54MM; LINK (none) -> https://www.digikey.de/product-detail/de/wurth-electronics-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; MANUFACTURER (none) -> Wurth Electronics Inc.; MANUFACTURERPARTNUMBER (none) -> 61300311121; POPULATED (none) -> TRUE; ROHSCERTIFICATE (none) -> Bleifrei / RoHS-konform; SOURCE (none) -> DIGIKEY; SOURCEPARTNUMBER (none) -> 732-5316-ND
- JP5, JP7: CLASS (none) -> CONNECTOR\JUMPER; DESCRIPTION (none) -> CONN HEADER VERT 2POS 2.54MM; LINK (none) -> https://www.digikey.de/product-detail/de/PREC002SAAN-RC/S10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; MANUFACTURER (none) -> Sullins Connector Solutions; MANUFACTURERPARTNUMBER (none) -> PREC002SAAN-RC; POPULATED (none) -> TRUE; ROHSCERTIFICATE (none) -> Bleifrei / RoHS-konform; SOURCE (none) -> DIGIKEY; SOURCEPARTNUMBER (none) -> S1012EC-02-ND
- JP6: CLASS (none) -> CONNECTOR\JUMPER; DESCRIPTION (none) -> CONN HEADER VERT 4POS 2.54MM; LINK (none) -> https://www.digikey.de/product-detail/de/sullins-connector-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; MANUFACTURER (none) -> Sullins Connector Solutions; MANUFACTURERPARTNUMBER (none) -> PRPC004SAAN-RC; POPULATED (none) -> TRUE; ROHSCERTIFICATE (none) -> Bleifrei / RoHS-konform; SOURCE (none) -> DIGIKEY; SOURCEPARTNUMBER (none) -> S1011EC-04-ND
- K1: CLASS (none) -> RELAY; DESCRIPTION (none) -> CONN PWR JACK 2.5X5.5MM SOLDER; LINK (none) -> http://www.digikey.de/product-detail/de/wurth-electronics-i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; MANUFACTURER (none) -> Wurth Electronics Inc.; MANUFACTURERPARTNUMBER (none) -> 694108106102; POPULATED (none) -> TRUE; ROHSCERTIFICATE (none) -> Bleifrei / RoHS-konform; SOURCE (none) -> DIGIKEY; SOURCEPARTNUMBER (none) -> 732-5933-1-ND
- LED1: CLASS (none) -> LED; DESCRIPTION (none) -> LED GREEN CLEAR 2PLCC SMD; LINK (none) -> https://www.digikey.de/product-detail/de/osram-opto-semicon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; MANUFACTURER (none) -> OSRAM Opto Semiconductors Inc.; MANUFACTURERPARTNUMBER (none) -> LG T67F-R1T1-24; POPULATED (none) -> TRUE; ROHSCERTIFICATE (none) -> Bleifrei / RoHS-konform; SOURCE (none) -> DIGIKEY; SOURCEPARTNUMBER (none) -> 475-3413-1-ND
- LED2: CLASS (none) -> LED; DESCRIPTION (none) -> LED YELLOW CLEAR 2PLCC SMD; LINK (none) -> https://www.digikey.de/product-detail/de/osram-opto-semicon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; MANUFACTURER (none) -> OSRAM Opto Semiconductors Inc.; MANUFACTURERPARTNUMBER (none) -> LY T676-S1T1-26-Z; POPULATED (none) -> TRUE; ROHSCERTIFICATE (none) -> Bleifrei / RoHS-konform; SOURCE (none) -> DIGIKEY; SOURCEPARTNUMBER (none) -> 475-2665-1-ND
- M1: CLASS (none) -> UNKNOWN CLASS; DESCRIPTION (none) -> NO DESCRIPTION; LINK (none) -> UNKNOWN LINK; MANUFACTURER (none) -> UNKNOWN MANUFACTURER; MANUFACTURERPARTNUMBER (none) -> UNKNOWN MANUFACTURER PART NUMBER; POPULATED (none) -> TRUE; ROHSCERTIFICATE (none) -> UNKNOWN ROHS CERTIFICATE; SOURCE (none) -> UNKNOWN SOURCE; SOURCEPARTNUMBER (none) -> UNKNOWN SOURCE PART NUMBER
- R1, R2, R3, R4: CLASS (none) -> RESISTOR; DESCRIPTION (none) -> RES 330K OHM 5%% 1/10W 0603; LINK (none) -> https://www.digikey.de/product-detail/de/stackpole-electron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; MANUFACTURER (none) -> Stackpole Electronics Inc; MANUFACTURERPARTNUMBER (none) -> RMCF0603JG330K; POPULATED (none) -> TRUE; ROHSCERTIFICATE (none) -> Bleifrei / RoHS-konform; SOURCE (none) -> DIGIKEY; SOURCEPARTNUMBER (none) -> RMCF0603JG330KCT-ND
- R10, R9: CLASS (none) -> RESISTOR; DESCRIPTION (none) -> RES 49.9 OHM 1%% 1/10W 0603; LINK (none) -> https://www.digikey.de/product-detail/de/stackpole-electron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; MANUFACTURER (none) -> Stackpole Electronics Inc; MANUFACTURERPARTNUMBER (none) -> RMCF0603FT49R9; POPULATED (none) -> TRUE; ROHSCERTIFICATE (none) -> Bleifrei / RoHS-konform; SOURCE (none) -> DIGIKEY; SOURCEPARTNUMBER (none) -> RMCF0603FT49R9CT-ND
- R11, R12: CLASS (none) -> RESISTOR; DESCRIPTION (none) -> RES 330 OHM 5%% 1/10W 0603; LINK (none) -> https://www.digikey.de/product-detail/de/stackpole-electron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; MANUFACTURER (none) -> Stackpole Electronics Inc; MANUFACTURERPARTNUMBER (none) -> RMCF0603JT330R; POPULATED (none) -> TRUE; ROHSCERTIFICATE (none) -> Bleifrei / RoHS-konform; SOURCE (none) -> DIGIKEY; SOURCEPARTNUMBER (none) -> RMCF0603JT330RCT-ND
- R5, R6, R7, R8: CLASS (none) -> RESISTOR; DESCRIPTION (none) -> RES 100 OHM 5%% 1/10W 0603; LINK (none) -> https://www.digikey.de/product-detail/de/stackpole-electron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; MANUFACTURER (none) -> Stackpole Electronics Inc; MANUFACTURERPARTNUMBER (none) -> RMCF0603JT100R; POPULATED (none) -> TRUE; ROHSCERTIFICATE (none) -> Bleifrei / RoHS-konform; SOURCE (none) -> DIGIKEY; SOURCEPARTNUMBER (none) -> RMCF0603JT100RCT-ND
- U1: CLASS (none) -> IC; DESCRIPTION (none) -> IC CLK BUFFER DVR 1:2 12MSOP; LINK (none) -> https://www.digikey.de/product-detail/de/linear-technology-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; MANUFACTURER (none) -> Linear Technology/Analog Devices; MANUFACTURERPARTNUMBER (none) -> LTC6957IMS-3#PBF; POPULATED (none) -> TRUE; ROHSCERTIFICATE (none) -> Bleifrei / RoHS-konform; SOURCE (none) -> DIGIKEY; SOURCEPARTNUMBER (none) -> LTC6957IMS-3#PBF-ND
- U2: CLASS (none) -> IC; DESCRIPTION (none) -> IC REG LINEAR 3V 200MA TSOT5; LINK (none) -> https://www.digikey.de/product-detail/de/analog-devices-inc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; MANUFACTURER (none) -> Analog Devices Inc.; MANUFACTURERPARTNUMBER (none) -> ADP151AUJZ-3.0-R7; POPULATED (none) -> TRUE; ROHSCERTIFICATE (none) -> Bleifrei / RoHS-konform; SOURCE (none) -> DIGIKEY; SOURCEPARTNUMBER (none) -> ADP151AUJZ-3.0-R7CT-ND
- X1, X2, X3, X4: CLASS (none) -> CONNECTOR; DESCRIPTION (none) -> CONN U.FL RCPT STR 50 OHM SMD; LINK (none) -> https://www.digikey.de/product-detail/de/hirose-electric-co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; MANUFACTURER (none) -> Hirose Electric Co Ltd; MANUFACTURERPARTNUMBER (none) -> U.FL-R-SMT(10); POPULATED (none) -> TRUE; ROHSCERTIFICATE (none) -> Bleifrei / RoHS-konform; SOURCE (none) -> DIGIKEY; SOURCEPARTNUMBER (none) -> H9161CT-ND
- X5, X6, X7, X8: CLASS (none) -> CONNECTOR; DESCRIPTION (none) -> CONN SMA JACK R/A 50 OHM PCB; LINK (none) -> https://www.digikey.de/product-detail/de/te-connectivity-am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; MANUFACTURER (none) -> TE Connectivity AMP Connectors; MANUFACTURERPARTNUMBER (none) -> 619540-1; POPULATED (none) -> TRUE; ROHSCERTIFICATE (none) -> Bleifrei / RoHS-konform; SOURCE (none) -> DIGIKEY; SOURCEPARTNUMBER (none) -> A120734-ND
