File: sc14dect-breakout/sc14cvm-evb.sch (EAGLE design)
At the start: 38 parts, among them K1 694108106102, U1 LDO-TLV1117, U2 LDO_EN-AP2127K, U3 SN74AVC4T245, X2 JACK2.5_SJ-2523, X3 JACK2.5_SJ-2523, X4 AUDIO, X5 DEBUG

Commit message: sc14cvm-evb: Add attributes
Parts:
- C1, C2, C3, C5, C6, C7, C8, C9: CLASS (none) -> CAPACITOR; DESCRIPTION (none) -> NO DESCRIPTION; LINK (none) -> UNKNOWN LINK; MANUFACTURER (none) -> UNKNOWN MANUFACTURER; MANUFACTURERPARTNUMBER (none) -> UNKNOWN MANUFACTURER PART NUMBER; POPULATED (none) -> TRUE; ROHSCERTIFICATE (none) -> UNKNOWN ROHS CERTIFICATE; SOURCE (none) -> UNKNOWN SOURCE; SOURCEPARTNUMBER (none) -> UNKNOWN SOURCE PART NUMBER
- C4: CLASS (none) -> CAPACITOR; DESCRIPTION (none) -> NO DESCRIPTION; LINK (none) -> https://www.digikey.de/product-detail/en/kemet/T495B107M010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; MANUFACTURER (none) -> UNKNOWN MANUFACTURER; MANUFACTURERPARTNUMBER (none) -> UNKNOWN MANUFACTURER PART NUMBER; POPULATED (none) -> TRUE; ROHSCERTIFICATE (none) -> UNKNOWN ROHS CERTIFICATE; SOURCE (none) -> UNKNOWN SOURCE; SOURCEPARTNUMBER (none) -> 399-18817-1-ND
- JP1, JP2: CLASS (none) -> CONNECTOR\JUMPER; DESCRIPTION (none) -> NO DESCRIPTION; LINK (none) -> https://www.digikey.de/product-detail/en/sullins-connector-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; MANUFACTURER (none) -> UNKNOWN MANUFACTURER; MANUFACTURERPARTNUMBER (none) -> UNKNOWN MANUFACTURER PART NUMBER; POPULATED (none) -> TRUE; ROHSCERTIFICATE (none) -> UNKNOWN ROHS CERTIFICATE; SOURCE (none) -> UNKNOWN SOURCE; SOURCEPARTNUMBER (none) -> UNKNOWN SOURCE PART NUMBER
- JP4: CLASS (none) -> CONNECTOR\JUMPER; DESCRIPTION (none) -> NO DESCRIPTION; LINK (none) -> UNKNOWN LINK; MANUFACTURER (none) -> UNKNOWN MANUFACTURER; MANUFACTURERPARTNUMBER (none) -> UNKNOWN MANUFACTURER PART NUMBER; POPULATED (none) -> TRUE; ROHSCERTIFICATE (none) -> UNKNOWN ROHS CERTIFICATE; SOURCE (none) -> UNKNOWN SOURCE; SOURCEPARTNUMBER (none) -> UNKNOWN SOURCE PART NUMBER
- K1: CLASS (none) -> RELAY; DESCRIPTION (none) -> NO DESCRIPTION; LINK (none) -> UNKNOWN LINK; MANUFACTURER (none) -> UNKNOWN MANUFACTURER; MANUFACTURERPARTNUMBER (none) -> UNKNOWN MANUFACTURER PART NUMBER; POPULATED (none) -> TRUE; ROHSCERTIFICATE (none) -> UNKNOWN ROHS CERTIFICATE; SOURCE (none) -> UNKNOWN SOURCE; SOURCEPARTNUMBER (none) -> UNKNOWN SOURCE PART NUMBER
- LED1: CLASS (none) -> LED; DESCRIPTION (none) -> NO DESCRIPTION; LINK (none) -> UNKNOWN LINK; MANUFACTURER (none) -> UNKNOWN MANUFACTURER; MANUFACTURERPARTNUMBER (none) -> UNKNOWN MANUFACTURER PART NUMBER; POPULATED (none) -> TRUE; ROHSCERTIFICATE (none) -> UNKNOWN ROHS CERTIFICATE; SOURCE (none) -> UNKNOWN SOURCE; SOURCEPARTNUMBER (none) -> UNKNOWN SOURCE PART NUMBER
- LED2: CLASS (none) -> LED; DESCRIPTION (none) -> NO DESCRIPTION; LINK (none) -> https://www.digikey.de/product-detail/en/LY+L29K-J1K2-26-Z/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; MANUFACTURER (none) -> UNKNOWN MANUFACTURER; MANUFACTURERPARTNUMBER (none) -> UNKNOWN MANUFACTURER PART NUMBER; POPULATED (none) -> TRUE; ROHSCERTIFICATE (none) -> UNKNOWN ROHS CERTIFICATE; SOURCE (none) -> UNKNOWN SOURCE; SOURCEPARTNUMBER (none) -> 475-2794-1-ND
- MOD1, TP1, TP2, TP3, TP4: CLASS (none) -> UNKNOWN CLASS; DESCRIPTION (none) -> NO DESCRIPTION; LINK (none) -> UNKNOWN LINK; MANUFACTURER (none) -> UNKNOWN MANUFACTURER; MANUFACTURERPARTNUMBER (none) -> UNKNOWN MANUFACTURER PART NUMBER; POPULATED (none) -> TRUE; ROHSCERTIFICATE (none) -> UNKNOWN ROHS CERTIFICATE; SOURCE (none) -> UNKNOWN SOURCE; SOURCEPARTNUMBER (none) -> UNKNOWN SOURCE PART NUMBER
- R1, R2, R3, R4, R5, R6: CLASS (none) -> RESISTOR; DESCRIPTION (none) -> NO DESCRIPTION; LINK (none) -> UNKNOWN LINK; MANUFACTURER (none) -> UNKNOWN MANUFACTURER; MANUFACTURERPARTNUMBER (none) -> UNKNOWN MANUFACTURER PART NUMBER; POPULATED (none) -> TRUE; ROHSCERTIFICATE (none) -> UNKNOWN ROHS CERTIFICATE; SOURCE (none) -> UNKNOWN SOURCE; SOURCEPARTNUMBER (none) -> UNKNOWN SOURCE PART NUMBER
- U1, U3: CLASS (none) -> IC; DESCRIPTION (none) -> NO DESCRIPTION; LINK (none) -> https://www.digikey.de/product-detail/en/texas-instruments/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; MANUFACTURER (none) -> UNKNOWN MANUFACTURER; MANUFACTURERPARTNUMBER (none) -> UNKNOWN MANUFACTURER PART NUMBER; POPULATED (none) -> TRUE; ROHSCERTIFICATE (none) -> UNKNOWN ROHS CERTIFICATE; SOURCE (none) -> UNKNOWN SOURCE; SOURCEPARTNUMBER (none) -> UNKNOWN SOURCE PART NUMBER
- U2: CLASS (none) -> IC; DESCRIPTION (none) -> NO DESCRIPTION; LINK (none) -> https://www.digikey.de/product-detail/en/AP2127K-1.8TRG1/AP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; MANUFACTURER (none) -> UNKNOWN MANUFACTURER; MANUFACTURERPARTNUMBER (none) -> AP2127K-1.8TRG1; POPULATED (none) -> TRUE; ROHSCERTIFICATE (none) -> UNKNOWN ROHS CERTIFICATE; SOURCE (none) -> UNKNOWN SOURCE; SOURCEPARTNUMBER (none) -> AP2127K-1.8TRG1DICT-ND
- X1, X2, X3, X5: CLASS (none) -> CONNECTOR; DESCRIPTION (none) -> NO DESCRIPTION; LINK (none) -> UNKNOWN LINK; MANUFACTURER (none) -> UNKNOWN MANUFACTURER; MANUFACTURERPARTNUMBER (none) -> UNKNOWN MANUFACTURER PART NUMBER; POPULATED (none) -> TRUE; ROHSCERTIFICATE (none) -> UNKNOWN ROHS CERTIFICATE; SOURCE (none) -> UNKNOWN SOURCE; SOURCEPARTNUMBER (none) -> UNKNOWN SOURCE PART NUMBER
- X4: CLASS (none) -> CONNECTOR; DESCRIPTION (none) -> NO DESCRIPTION; LINK (none) -> https://www.digikey.de/product-detail/en/PRPC005DAAN-RC/S20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; MANUFACTURER (none) -> UNKNOWN MANUFACTURER; MANUFACTURERPARTNUMBER (none) -> UNKNOWN MANUFACTURER PART NUMBER; POPULATED (none) -> TRUE; ROHSCERTIFICATE (none) -> UNKNOWN ROHS CERTIFICATE; SOURCE (none) -> UNKNOWN SOURCE; SOURCEPARTNUMBER (none) -> UNKNOWN SOURCE PART NUMBER
