File: siu-clock-breakout/siu-clock-breakout.brd (EAGLE design)
At the start: 50 x 100 mm, 32 parts, among them IC1 ISL83485, IC2 ISL83485, IC3 ISL83485, M1 MENTOR_12701001, T1 BC847, U1 LDO-TLV1117

Commit message: siu-clock-breakout: Add missing component values
Parts:
- C1, C2, C3: value (none) -> 100n
- R10, R4: value (none) -> 330
Changed lines of the file:
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@@
 <attribute name="MF" value="" x="35.56" y="34.29" size="1.778" layer="27" rot="R90" display="off"/>
 </element>
-<element name="C1" library="rc-sysmocom" package="_0603" value="" x="32.004" y="13.716" smashed="yes" rot="R180">
+<element name="C1" library="rc-sysmocom" package="_0603" value="100n" x="32.004" y="13.716" smashed="yes" rot="R180">
 <attribute name="NAME" x="30.1625" y="14.6685" size="1.016" layer="25" font="vector" ratio="14"/>
 <attribute name="VALUE" x="33.5915" y="15.2083" size="0.508" layer="27" font="vector" ratio="10" rot="R180"/>
 </element>
-<element name="C2" library="rc-sysmocom" package="_0603" value="" x="32.004" y="22.352" rot="R180"/>
-<element name="C3" library="rc-sysmocom" package="_0603" value="" x="32.004" y="30.988" rot="R180"/>
+<element name="C2" library="rc-sysmocom" package="_0603" value="100n" x="32.004" y="22.352" rot="R180"/>
+<element name="C3" library="rc-sysmocom" package="_0603" value="100n" x="32.004" y="30.988" rot="R180"/>
 <element name="R1" library="rc-sysmocom" package="_0805" value="120" x="27.94" y="17.018" rot="R270"/>
 <element name="R2" library="rc-sysmocom" package="_0805" value="DNP" x="29.21" y="25.654" rot="R270"/>
@@
 <element name="C5" library="rc-sysmocom" package="CPOL1206" value="10-100u / 6.3V" x="39.624" y="6.604" rot="R270"/>
 <element name="LED1" library="LED-PLCC2" package="PLCC2-MIN" value="LEDPLCC2-MIN" x="13.716" y="8.382" rot="R180"/>
-<element name="R4" library="rc-sysmocom" package="_0603" value="" x="26.416" y="5.08" smashed="yes">
+<element name="R4" library="rc-sysmocom" package="_0603" value="330" x="26.416" y="5.08" smashed="yes">
 <attribute name="NAME" x="24.7015" y="5.6515" size="1.016" layer="25" font="vector" ratio="14" rot="R180"/>
 <attribute name="VALUE" x="24.8285" y="3.5877" size="0.508" layer="27" font="vector" ratio="10"/>
@@
 <attribute name="SOURCE" value="DIGIKEY" x="14.224" y="49.53" size="1.778" layer="27" font="vector" ratio="14" rot="R180" display="off"/>
 </element>
-<element name="R10" library="rc-sysmocom" package="_0603" value="" x="26.416" y="3.81" smashed="yes">
+<element name="R10" library="rc-sysmocom" package="_0603" value="330" x="26.416" y="3.81" smashed="yes">
 <attribute name="NAME" x="24.7015" y="4.1275" size="1.016" layer="25" font="vector" ratio="14" rot="R180"/>
 <attribute name="VALUE" x="24.8285" y="2.3177" size="0.508" layer="27" font="vector" ratio="10"/>
