File: sfp-breakout/sfp-experimenter.sch (EAGLE design)
At the start: 51 parts, among them IC1 SN65LVDS1DBV, IC2 SN65LVDT2DBV, J1 PJ-002BH-SMT-TR, T1 BC847, T2 BC847, U1 LDO-MCP1825S, X1 PINHD-1X5LOCK, X2 PINHD-1X5LOCK, X3 PINHD-1X4LOCK

Commit message: sfp-experimnter: update extd attribs on D1, D2 to avail types
Parts:
- C6, R1, R10, R12, R2, R3, R4, R5, R7, R8, R9: ROHSCERTIFICATE UNKNOWN ROHS CERTIFICATE -> RoHS3-konform
- D1: DESCRIPTION DIODE SCHOTTKY 60V 1A SMA -> DIODE SCHOTTKY 60V 2A SMA; LINK http://www.digikey.de/product-detail/de/SS16T3G/SS16T3GOSCT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 -> https://www.digikey.de/product-detail/de/stmicroelectronics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; MANUFACTURER ON Semiconductor -> STMicroelectronics; MANUFACTURERPARTNUMBER SS16T3G -> STPS2L60A; ROHSCERTIFICATE Bleifrei / RoHS-konform -> RoHS3-konform; SOURCEPARTNUMBER SS16T3GOSCT-ND -> 497-2461-1-ND
- D2: DESCRIPTION TVS DIODE 5V 9.2V DO214AC -> TVS DIODE 5VWM 9.2VC SMA; LINK https://www.digikey.de/product-detail/de/wurth-electronics-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 -> https://www.digikey.de/product-detail/de/bourns-inc/SMAJ5-0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; MANUFACTURER Wurth Electronics Inc. -> Bourns Inc.; MANUFACTURERPARTNUMBER 824500500 -> SMAJ5.0A; ROHSCERTIFICATE Bleifrei / RoHS-konform -> RoHS3-konform; SOURCEPARTNUMBER 732-9974-1-ND -> SMAJ5.0ABCT-ND
- J1, L1, L2: ROHSCERTIFICATE UNKNOWN ROHS CERTIFICATE -> RoHS-konform
Changed lines of the file:
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@@
 <attribute name="MANUFACTURERPARTNUMBER" value="AIMC-0603-1N0S-T"/>
 <attribute name="POPULATED" value="TRUE"/>
-<attribute name="ROHSCERTIFICATE" value="UNKNOWN ROHS CERTIFICATE"/>
+<attribute name="ROHSCERTIFICATE" value="RoHS-konform"/>
 <attribute name="SOURCE" value="DIGIKEY"/>
 <attribute name="SOURCEPARTNUMBER" value="535-11529-1-ND"/>
@@
 <attribute name="MANUFACTURERPARTNUMBER" value="AIMC-0603-1N0S-T"/>
 <attribute name="POPULATED" value="TRUE"/>
-<attribute name="ROHSCERTIFICATE" value="UNKNOWN ROHS CERTIFICATE"/>
+<attribute name="ROHSCERTIFICATE" value="RoHS-konform"/>
 <attribute name="SOURCE" value="DIGIKEY"/>
 <attribute name="SOURCEPARTNUMBER" value="535-11529-1-ND"/>
@@
 <attribute name="MANUFACTURERPARTNUMBER" value="T520C107M006ATE045"/>
 <attribute name="POPULATED" value="TRUE"/>
-<attribute name="ROHSCERTIFICATE" value="UNKNOWN ROHS CERTIFICATE"/>
+<attribute name="ROHSCERTIFICATE" value="RoHS3-konform"/>
 <attribute name="SOURCE" value="DIGIKEY"/>
 <attribute name="SOURCEPARTNUMBER" value="399-4658-1-ND"/>
@@
 <attribute name="MANUFACTURERPARTNUMBER" value="PJ-002BH-SMT-TR"/>
 <attribute name="POPULATED" value="TRUE"/>
-<attribute name="ROHSCERTIFICATE" value="UNKNOWN ROHS CERTIFICATE"/>
+<attribute name="ROHSCERTIFICATE" value="RoHS-konform"/>
 <attribute name="SOURCE" value="DIGIKEY"/>
 <attribute name="SOURCEPARTNUMBER" value="CP-002BHPJCT-ND"/>
@@
 <attribute name="MANUFACTURERPARTNUMBER" value="RC0603FR-0710KL"/>
 <attribute name="POPULATED" value="TRUE"/>
-<attribute name="ROHSCERTIFICATE" value="UNKNOWN ROHS CERTIFICATE"/>
+<attribute name="ROHSCERTIFICATE" value="RoHS3-konform"/>
 <attribute name="SOURCE" value="DIGIKEY"/>
 <attribute name="SOURCEPARTNUMBER" value="311-10.0KHRCT-ND"/>
@@
 <attribute name="MANUFACTURERPARTNUMBER" value="RC0603FR-0710KL"/>
 <attribute name="POPULATED" value="TRUE"/>
-<attribute name="ROHSCERTIFICATE" value="UNKNOWN ROHS CERTIFICATE"/>
+<attribute name="ROHSCERTIFICATE" value="RoHS3-konform"/>
 <attribute name="SOURCE" value="DIGIKEY"/>
 <attribute name="SOURCEPARTNUMBER" value="311-10.0KHRCT-ND"/>
@@
 <attribute name="MANUFACTURERPARTNUMBER" value="RC0603FR-0710KL"/>
 <attribute name="POPULATED" value="TRUE"/>
-<attribute name="ROHSCERTIFICATE" value="UNKNOWN ROHS CERTIFICATE"/>
+<attribute name="ROHSCERTIFICATE" value="RoHS3-konform"/>
 <attribute name="SOURCE" value="DIGIKEY"/>
 <attribute name="SOURCEPARTNUMBER" value="311-10.0KHRCT-ND"/>
@@
 <attribute name="MANUFACTURERPARTNUMBER" value="RC0603FR-0710KL"/>
 <attribute name="POPULATED" value="TRUE"/>
-<attribute name="ROHSCERTIFICATE" value="UNKNOWN ROHS CERTIFICATE"/>
+<attribute name="ROHSCERTIFICATE" value="RoHS3-konform"/>
 <attribute name="SOURCE" value="DIGIKEY"/>
 <attribute name="SOURCEPARTNUMBER" value="311-10.0KHRCT-ND"/>
@@
 <attribute name="MANUFACTURERPARTNUMBER" value="RC0603FR-0710KL"/>
 <attribute name="POPULATED" value="TRUE"/>
-<attribute name="ROHSCERTIFICATE" value="UNKNOWN ROHS CERTIFICATE"/>
+<attribute name="ROHSCERTIFICATE" value="RoHS3-konform"/>
 <attribute name="SOURCE" value="DIGIKEY"/>
 <attribute name="SOURCEPARTNUMBER" value="311-10.0KHRCT-ND"/>
@@
 <part name="D1" library="sfp-experimenter" deviceset="DIODE-SCHOTTKY" device="-SMA" value="SS16T3G">
 <attribute name="CLASS" value="DIODE"/>
-<attribute name="DESCRIPTION" value="DIODE SCHOTTKY 60V 1A SMA"/>
-<attribute name="LINK" value="http://www.digikey.de/product-detail/de/SS16T3G/SS16T3GOSCT-ND/964637"/>
-<attribute name="MANUFACTURER" value="ON Semiconductor"/>
-<attribute name="MANUFACTURERPARTNUMBER" value="SS16T3G"/>
-<attribute name="POPULATED" value="TRUE"/>
-<attribute name="ROHSCERTIFICATE" value="Bleifrei / RoHS-konform"/>
-<attribute name="SOURCE" value="DIGIKEY"/>
-<attribute name="SOURCEPARTNUMBER" value="SS16T3GOSCT-ND"/>
+<attribute name="DESCRIPTION" value="DIODE SCHOTTKY 60V 2A SMA"/>
+<attribute name="LINK" value="https://www.digikey.de/product-detail/de/stmicroelectronics/STPS2L60A/497-2461-1-ND"/>
+<attribute name="MANUFACTURER" value="STMicroelectronics"/>
+<attribute name="MANUFACTURERPARTNUMBER" value="STPS2L60A"/>
+<attribute name="POPULATED" value="TRUE"/>
+<attribute name="ROHSCERTIFICATE" value="RoHS3-konform"/>
+<attribute name="SOURCE" value="DIGIKEY"/>
+<attribute name="SOURCEPARTNUMBER" value="497-2461-1-ND"/>
 </part>
 <part name="D2" library="sfp-experimenter" deviceset="DIODE-TVS" device="-SMA" value="824500500">
 <attribute name="CLASS" value="DIODE"/>
-<attribute name="DESCRIPTION" value="TVS DIODE 5V 9.2V DO214AC"/>
-<attribute name="LINK" value="https://www.digikey.de/product-detail/de/wurth-electronics-inc/824500500/732-9974-1-ND/5871127"/>
-<attribute name="MANUFACTURER" value="Wurth Electronics Inc."/>
-<attribute name="MANUFACTURERPARTNUMBER" value="824500500"/>
-<attribute name="POPULATED" value="TRUE"/>
-<attribute name="ROHSCERTIFICATE" value="Bleifrei / RoHS-konform"/>
-<attribute name="SOURCE" value="DIGIKEY"/>
-<attribute name="SOURCEPARTNUMBER" value="732-9974-1-ND"/>
+<attribute name="DESCRIPTION" value="TVS DIODE 5VWM 9.2VC SMA"/>
+<attribute name="LINK" value="https://www.digikey.de/product-detail/de/bourns-inc/SMAJ5-0A/SMAJ5-0ABCT-ND/2254241"/>
+<attribute name="MANUFACTURER" value="Bourns Inc."/>
+<attribute name="MANUFACTURERPARTNUMBER" value="SMAJ5.0A"/>
+<attribute name="POPULATED" value="TRUE"/>
+<attribute name="ROHSCERTIFICATE" value="RoHS3-konform"/>
+<attribute name="SOURCE" value="DIGIKEY"/>
+<attribute name="SOURCEPARTNUMBER" value="SMAJ5.0ABCT-ND"/>
 </part>
 <part name="R6" library="sfp-experimenter" deviceset="RESISTOR" device="_0402" value="DNP">
@@
 <attribute name="MANUFACTURERPARTNUMBER" value="RC0603FR-0710KL"/>
 <attribute name="POPULATED" value="TRUE"/>
-<attribute name="ROHSCERTIFICATE" value="UNKNOWN ROHS CERTIFICATE"/>
+<attribute name="ROHSCERTIFICATE" value="RoHS3-konform"/>
 <attribute name="SOURCE" value="DIGIKEY"/>
 <attribute name="SOURCEPARTNUMBER" value="311-10.0KHRCT-ND"/>
@@
 <attribute name="MANUFACTURERPARTNUMBER" value="ERJ-3GEYJ331V"/>
 <attribute name="POPULATED" value="TRUE"/>
-<attribute name="ROHSCERTIFICATE" value="UNKNOWN ROHS CERTIFICATE"/>
+<attribute name="ROHSCERTIFICATE" value="RoHS3-konform"/>
 <attribute name="SOURCE" value="DIGIKEY"/>
 <attribute name="SOURCEPARTNUMBER" value="P330GCT-ND"/>
@@
 <attribute name="MANUFACTURERPARTNUMBER" value="RC0603FR-0710KL"/>
 <attribute name="POPULATED" value="TRUE"/>
-<attribute name="ROHSCERTIFICATE" value="UNKNOWN ROHS CERTIFICATE"/>
+<attribute name="ROHSCERTIFICATE" value="RoHS3-konform"/>
 <attribute name="SOURCE" value="DIGIKEY"/>
 <attribute name="SOURCEPARTNUMBER" value="311-10.0KHRCT-ND"/>
@@
 <attribute name="MANUFACTURERPARTNUMBER" value="ERJ-3GEYJ331V"/>
 <attribute name="POPULATED" value="TRUE"/>
-<attribute name="ROHSCERTIFICATE" value="UNKNOWN ROHS CERTIFICATE"/>
+<attribute name="ROHSCERTIFICATE" value="RoHS3-konform"/>
 <attribute name="SOURCE" value="DIGIKEY"/>
 <attribute name="SOURCEPARTNUMBER" value="P330GCT-ND"/>
@@
 <attribute name="MANUFACTURERPARTNUMBER" value="RK73H1JTTD1003F"/>
 <attribute name="POPULATED" value="TRUE"/>
-<attribute name="ROHSCERTIFICATE" value="UNKNOWN ROHS CERTIFICATE"/>
+<attribute name="ROHSCERTIFICATE" value="RoHS3-konform"/>
 <attribute name="SOURCE" value="DIGIKEY"/>
 <attribute name="SOURCEPARTNUMBER" value="2019-RK73H1JTTD1003FCT-ND"/>
@@
 </instance>
 <instance part="D2" gate="G$1" x="68.58" y="76.2" rot="R90">
-<attribute name="DESCRIPTION" x="68.58" y="76.2" size="1.778" layer="96" rot="R90" display="off"/>
-<attribute name="MANUFACTURER" x="68.58" y="76.2" size="1.778" layer="96" rot="R90" display="off"/>
-<attribute name="MANUFACTURERPARTNUMBER" x="68.58" y="76.2" size="1.778" layer="96" rot="R90" display="off"/>
-<attribute name="SOURCE" x="68.58" y="76.2" size="1.778" layer="96" rot="R90" display="off"/>
-<attribute name="SOURCEPARTNUMBER" x="68.58" y="76.2" size="1.778" layer="96" rot="R90" display="off"/>
-<attribute name="ROHSCERTIFICATE" x="68.58" y="76.2" size="1.778" layer="96" rot="R90" display="off"/>
-<attribute name="POPULATED" x="68.58" y="76.2" size="1.778" layer="96" rot="R90" display="off"/>
-<attribute name="CLASS" x="68.58" y="76.2" size="1.778" layer="96" rot="R90" display="off"/>
-<attribute name="LINK" x="68.58" y="76.2" size="1.778" layer="96" rot="R90" display="off"/>
+<attribute name="DESCRIPTION" x="68.58" y="76.2" size="1.778" layer="96" display="off"/>
+<attribute name="MANUFACTURER" x="68.58" y="76.2" size="1.778" layer="96" display="off"/>
+<attribute name="MANUFACTURERPARTNUMBER" x="68.58" y="76.2" size="1.778" layer="96" display="off"/>
+<attribute name="SOURCE" x="68.58" y="76.2" size="1.778" layer="96" display="off"/>
+<attribute name="SOURCEPARTNUMBER" x="68.58" y="76.2" size="1.778" layer="96" display="off"/>
+<attribute name="ROHSCERTIFICATE" x="68.58" y="76.2" size="1.778" layer="96" display="off"/>
+<attribute name="POPULATED" x="68.58" y="76.2" size="1.778" layer="96" display="off"/>
+<attribute name="CLASS" x="68.58" y="76.2" size="1.778" layer="96" display="off"/>
+<attribute name="LINK" x="68.58" y="76.2" size="1.778" layer="96" display="off"/>
 </instance>
 <instance part="R6" gate="G$1" x="144.78" y="129.54" rot="R270">

Commit message: sfp-*: change all 10µF/16V 0805 to 1206 (solves SYS#5397)
also update all URLs to the current Digikey URI scheme
Parts:
- C1, C3, C9: DATASHEET (none) -> https://www.samsungsem.com/kr/support/product-search/mlcc/C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; DESCRIPTION CAP CER 10UF 16V X5R 0805 -> CAP CER 10UF 16V X5R 1206; LINK https://www.digikey.de/product-detail/de/samsung-electro-me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 -> https://www.digikey.com/en/products/detail/samsung-electro-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; MANUFACTURERPARTNUMBER CL21A106KOCLRNC -> CL31A106KOHNNNE; ROHSCERTIFICATE Bleifrei / RoHS-konform -> ROHS3 Compliant; SOURCEPARTNUMBER 1276-2399-1-ND -> 1276-1137-1-ND
- C10, C14, C2, C4, C5, C7, C8: DATASHEET (none) -> http://www.samsungsem.com/kr/support/product-search/mlcc/CL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; LINK http://www.digikey.de/product-detail/de/foo/1276-1005-1-ND -> https://www.digikey.com/product-detail/en/samsung-electro-m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; ROHSCERTIFICATE Bleifrei / RoHS-konform -> ROHS3 Compliant
- C11, C15: DATASHEET (none) -> https://datasheets.avx.com/X7RDielectric.pdf; LINK https://www.digikey.de/product-detail/de/avx-corporation/06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 -> https://www.digikey.com/product-detail/en/avx-corporation/0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; ROHSCERTIFICATE Bleifrei / RoHS-konform -> ROHS3 Compliant
- C12, C16: DATASHEET (none) -> https://www.yageo.com/upload/media/product/productsearch/da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; LINK https://www.digikey.de/product-detail/de/yageo/CC0603KRX7R9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 -> https://www.digikey.com/product-detail/en/yageo/CC0603KRX7R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; ROHSCERTIFICATE Bleifrei / RoHS-konform -> ROHS3 Compliant
- C13, C17: DATASHEET (none) -> https://www.yageo.com/upload/media/product/productsearch/da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; LINK https://www.digikey.de/product-detail/de/yageo/CC0603JRNPO9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 -> https://www.digikey.com/product-detail/en/yageo/CC0603JRNPO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; ROHSCERTIFICATE Bleifrei / RoHS-konform -> ROHS3 Compliant
- C6: DATASHEET (none) -> https://content.kemet.com/datasheets/KEM_T2076_T52X-530.pdf; LINK https://www.digikey.de/product-detail/de/kemet/T520C107M006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 -> https://www.digikey.com/product-detail/en/kemet/T520C107M00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; ROHSCERTIFICATE RoHS3-konform -> ROHS3 Compliant
- D1: DATASHEET (none) -> https://www.st.com/content/ccc/resource/technical/document/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; LINK https://www.digikey.de/product-detail/de/stmicroelectronics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 -> https://www.digikey.com/en/products/detail/stmicroelectroni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; ROHSCERTIFICATE RoHS3-konform -> ROHS3 Compliant
- D2: DATASHEET (none) -> https://www.bourns.com/docs/Product-Datasheets/SMAJ.pdf; LINK https://www.digikey.de/product-detail/de/bourns-inc/SMAJ5-0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 -> https://www.digikey.com/en/products/detail/bourns-inc/SMAJ5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; ROHSCERTIFICATE RoHS3-konform -> ROHS3 Compliant
- IC1: DATASHEET (none) -> http://www.ti.com/general/docs/suppproductinfo.tsp?distId=1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; DESCRIPTION IC 1/0 DRIVER LVDS SOT23-5 -> IC DRIVER 1/0 SOT23-5; LINK https://www.digikey.de/product-detail/de/texas-instruments/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 -> https://www.digikey.com/product-detail/en/texas-instruments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; ROHSCERTIFICATE Bleifrei / RoHS-konform -> ROHS3 Compliant
- IC2: DATASHEET (none) -> http://www.ti.com/general/docs/suppproductinfo.tsp?distId=1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; DESCRIPTION IC DIFF LINE RECEIVER SOT-23-5 -> IC RECEIVER 0/1 SOT23-5; LINK https://www.digikey.de/product-detail/de/texas-instruments/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 -> https://www.digikey.com/product-detail/en/texas-instruments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; ROHSCERTIFICATE Bleifrei / RoHS-konform -> ROHS3 Compliant
- J1: DATASHEET (none) -> https://www.cuidevices.com/product/resource/pj-002bh-smt-tr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; LINK https://www.digikey.de/product-detail/de/cui-inc/PJ-002BH-S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 -> https://www.digikey.com/product-detail/en/cui-devices/PJ-00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; ROHSCERTIFICATE RoHS-konform -> RoHS Compliant
- L1, L2: DATASHEET (none) -> https://abracon.com/Magnetics/new/AIMC-0603.pdf; LINK https://www.digikey.de/product-detail/de/abracon-llc/AIMC-0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 -> https://www.digikey.com/product-detail/en/abracon-llc/AIMC-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; ROHSCERTIFICATE RoHS-konform -> RoHS Compliant
- R1, R2, R3, R4, R5, R7, R8: DATASHEET (none) -> https://www.yageo.com/upload/media/product/productsearch/da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; DESCRIPTION RES SMD 10K OHM 1%% 1/10W 0603 -> RES 10K OHM 1% 1/10W 0603; LINK https://www.digikey.de/product-detail/de/yageo/RC0603FR-071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 -> https://www.digikey.com/en/products/detail/yageo/RC0603FR-0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; MANUFACTURER Yageo -> YAGEO; ROHSCERTIFICATE RoHS3-konform -> ROHS3 Compliant
- R10, R9: DATASHEET (none) -> https://industrial.panasonic.com/ww/products/resistors/chip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; DESCRIPTION RES SMD 330 OHM 5%% 1/10W 0603 -> RES SMD 330 OHM 5% 1/10W 0603; LINK https://www.digikey.de/product-detail/de/panasonic-electron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 -> https://www.digikey.com/product-detail/en/panasonic-electro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; ROHSCERTIFICATE RoHS3-konform -> ROHS3 Compliant
- R12: DATASHEET (none) -> https://www.koaspeer.com/pdfs/RK73H.pdf; DESCRIPTION RES 100K OHM 1%% 1/10W 0603 -> RES 100K OHM 1% 1/10W 0603; LINK https://www.digikey.de/product-detail/de/koa-speer-electron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 -> https://www.digikey.com/product-detail/en/koa-speer-electro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; ROHSCERTIFICATE RoHS3-konform -> ROHS3 Compliant
- SFP1: DATASHEET (none) -> https://media.digikey.com/pdf/Data%20Sheets/Amphenol%20PDFs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; LINK https://www.digikey.de/product-detail/de/amphenol-icc-comme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 -> https://www.digikey.com/product-detail/en/amphenol-icc-comm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; ROHSCERTIFICATE Bleifrei / RoHS-konform -> RoHS Compliant
- U1: DATASHEET (none) -> https://ww1.microchip.com/downloads/en/DeviceDoc/22056b.pdf; LINK https://www.digikey.de/product-detail/de/microchip-technolo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 -> https://www.digikey.com/en/products/detail/microchip-techno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; ROHSCERTIFICATE Bleifrei / RoHS-konform -> ROHS3 Compliant
