File: sfp-breakout/sfp-breakout.sch (EAGLE design)
At the start: 40 parts, among them J1 PJ-002BH-SMT-TR, T1 BC847, T2 BC847, U1 LDO-MCP1825S, X1 PINHD-1X5LOCK, X2 PINHD-1X5LOCK, X3 PINHD-1X4LOCK

Commit message: sfp-*: change all 10µF/16V 0805 to 1206 (solves SYS#5397)
also update all URLs to the current Digikey URI scheme
Parts:
- C6: DESCRIPTION CAP TANT 100UF 10%% 6.3V 2312 -> CAP TANT 100UF 10% 6.3V 2312
Changed lines of the file:
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@@
 <grid distance="0.1" unitdist="inch" unit="inch" style="lines" multiple="1" display="no" altdistance="0.01" altunitdist="inch" altunit="inch"/>
 <layers>
-<layer number="1" name="Top" color="4" fill="1" visible="yes" active="no"/>
-<layer number="2" name="Route2" color="14" fill="3" visible="yes" active="no"/>
-<layer number="3" name="Route3" color="4" fill="3" visible="yes" active="no"/>
-<layer number="4" name="Route4" color="1" fill="4" visible="yes" active="no"/>
-<layer number="5" name="Route5" color="4" fill="4" visible="yes" active="no"/>
-<layer number="6" name="Route6" color="1" fill="8" visible="yes" active="no"/>
-<layer number="7" name="Route7" color="4" fill="8" visible="yes" active="no"/>
-<layer number="8" name="Route8" color="1" fill="2" visible="yes" active="no"/>
-<layer number="9" name="Route9" color="4" fill="2" visible="yes" active="no"/>
-<layer number="10" name="Route10" color="1" fill="7" visible="yes" active="no"/>
-<layer number="11" name="Route11" color="4" fill="7" visible="yes" active="no"/>
-<layer number="12" name="Route12" color="1" fill="5" visible="yes" active="no"/>
-<layer number="13" name="Route13" color="4" fill="5" visible="yes" active="no"/>
-<layer number="14" name="Route14" color="1" fill="6" visible="yes" active="no"/>
-<layer number="15" name="Route15" color="11" fill="6" visible="yes" active="no"/>
-<layer number="16" name="Bottom" color="1" fill="1" visible="yes" active="no"/>
-<layer number="17" name="Pads" color="2" fill="1" visible="yes" active="no"/>
-<layer number="18" name="Vias" color="2" fill="1" visible="yes" active="no"/>
-<layer number="19" name="Unrouted" color="6" fill="1" visible="yes" active="no"/>
-<layer number="20" name="Dimension" color="15" fill="1" visible="yes" active="no"/>
-<layer number="21" name="tPlace" color="7" fill="1" visible="yes" active="no"/>
-<layer number="22" name="bPlace" color="7" fill="1" visible="yes" active="no"/>
-<layer number="23" name="tOrigins" color="15" fill="1" visible="yes" active="no"/>
-<layer number="24" name="bOrigins" color="15" fill="1" visible="yes" active="no"/>
-<layer number="25" name="tNames" color="7" fill="1" visible="yes" active="no"/>
-<layer number="26" name="bNames" color="7" fill="1" visible="yes" active="no"/>
-<layer number="27" name="tValues" color="7" fill="1" visible="yes" active="no"/>
-<layer number="28" name="bValues" color="7" fill="1" visible="yes" active="no"/>
+<layer number="1" name="Top" color="4" fill="1" visible="no" active="no"/>
+<layer number="2" name="Route2" color="14" fill="3" visible="no" active="no"/>
+<layer number="3" name="Route3" color="4" fill="3" visible="no" active="no"/>
+<layer number="4" name="Route4" color="1" fill="4" visible="no" active="no"/>
+<layer number="5" name="Route5" color="4" fill="4" visible="no" active="no"/>
+<layer number="6" name="Route6" color="1" fill="8" visible="no" active="no"/>
+<layer number="7" name="Route7" color="4" fill="8" visible="no" active="no"/>
+<layer number="8" name="Route8" color="1" fill="2" visible="no" active="no"/>
+<layer number="9" name="Route9" color="4" fill="2" visible="no" active="no"/>
+<layer number="10" name="Route10" color="1" fill="7" visible="no" active="no"/>
+<layer number="11" name="Route11" color="4" fill="7" visible="no" active="no"/>
+<layer number="12" name="Route12" color="1" fill="5" visible="no" active="no"/>
+<layer number="13" name="Route13" color="4" fill="5" visible="no" active="no"/>
+<layer number="14" name="Route14" color="1" fill="6" visible="no" active="no"/>
+<layer number="15" name="Route15" color="11" fill="6" visible="no" active="no"/>
+<layer number="16" name="Bottom" color="1" fill="1" visible="no" active="no"/>
+<layer number="17" name="Pads" color="2" fill="1" visible="no" active="no"/>
+<layer number="18" name="Vias" color="2" fill="1" visible="no" active="no"/>
+<layer number="19" name="Unrouted" color="6" fill="1" visible="no" active="no"/>
+<layer number="20" name="Dimension" color="15" fill="1" visible="no" active="no"/>
+<layer number="21" name="tPlace" color="7" fill="1" visible="no" active="no"/>
+<layer number="22" name="bPlace" color="7" fill="1" visible="no" active="no"/>
+<layer number="23" name="tOrigins" color="15" fill="1" visible="no" active="no"/>
+<layer number="24" name="bOrigins" color="15" fill="1" visible="no" active="no"/>
+<layer number="25" name="tNames" color="7" fill="1" visible="no" active="no"/>
+<layer number="26" name="bNames" color="7" fill="1" visible="no" active="no"/>
+<layer number="27" name="tValues" color="7" fill="1" visible="no" active="no"/>
+<layer number="28" name="bValues" color="7" fill="1" visible="no" active="no"/>
 <layer number="29" name="tStop" color="7" fill="3" visible="no" active="no"/>
 <layer number="30" name="bStop" color="7" fill="6" visible="no" active="no"/>
@@
 <layer number="35" name="tGlue" color="7" fill="4" visible="no" active="no"/>
 <layer number="36" name="bGlue" color="7" fill="5" visible="no" active="no"/>
-<layer number="37" name="tTest" color="7" fill="1" visible="yes" active="no"/>
-<layer number="38" name="bTest" color="7" fill="1" visible="yes" active="no"/>
+<layer number="37" name="tTest" color="7" fill="1" visible="no" active="no"/>
+<layer number="38" name="bTest" color="7" fill="1" visible="no" active="no"/>
 <layer number="39" name="tKeepout" color="4" fill="11" visible="no" active="no"/>
 <layer number="40" name="bKeepout" color="1" fill="11" visible="no" active="no"/>
@@
 <layer number="44" name="Drills" color="7" fill="1" visible="no" active="no"/>
 <layer number="45" name="Holes" color="7" fill="1" visible="no" active="no"/>
-<layer number="46" name="Milling" color="3" fill="1" visible="yes" active="no"/>
-<layer number="47" name="Measures" color="7" fill="1" visible="yes" active="no"/>
-<layer number="48" name="Document" color="7" fill="1" visible="yes" active="no"/>
-<layer number="49" name="Reference" color="7" fill="1" visible="yes" active="no"/>
-<layer number="50" name="dxf" color="7" fill="1" visible="yes" active="no"/>
-<layer number="51" name="tDocu" color="7" fill="1" visible="yes" active="no"/>
-<layer number="52" name="bDocu" color="7" fill="1" visible="yes" active="no"/>
-<layer number="53" name="tGND_GNDA" color="7" fill="9" visible="yes" active="no"/>
-<layer number="54" name="bGND_GNDA" color="1" fill="9" visible="yes" active="no"/>
-<layer number="56" name="wert" color="7" fill="1" visible="yes" active="no"/>
-<layer number="57" name="tCAD" color="6" fill="1" visible="yes" active="no"/>
-<layer number="59" name="tMark" color="7" fill="1" visible="yes" active="no"/>
-<layer number="60" name="bMark" color="7" fill="1" visible="yes" active="no"/>
+<layer number="46" name="Milling" color="3" fill="1" visible="no" active="no"/>
+<layer number="47" name="Measures" color="7" fill="1" visible="no" active="no"/>
+<layer number="48" name="Document" color="7" fill="1" visible="no" active="no"/>
+<layer number="49" name="Reference" color="7" fill="1" visible="no" active="no"/>
+<layer number="50" name="dxf" color="7" fill="1" visible="no" active="no"/>
+<layer number="51" name="tDocu" color="7" fill="1" visible="no" active="no"/>
+<layer number="52" name="bDocu" color="7" fill="1" visible="no" active="no"/>
+<layer number="53" name="tGND_GNDA" color="7" fill="9" visible="no" active="no"/>
+<layer number="54" name="bGND_GNDA" color="1" fill="9" visible="no" active="no"/>
+<layer number="56" name="wert" color="7" fill="1" visible="no" active="no"/>
+<layer number="57" name="tCAD" color="6" fill="1" visible="no" active="no"/>
+<layer number="59" name="tMark" color="7" fill="1" visible="no" active="no"/>
+<layer number="60" name="bMark" color="7" fill="1" visible="no" active="no"/>
 <layer number="90" name="Modules" color="5" fill="1" visible="yes" active="yes"/>
 <layer number="91" name="Nets" color="2" fill="1" visible="yes" active="yes"/>
@@
 <part name="C6" library="rcl" deviceset="CPOL-EU" device="CT6032" value="100u">
 <attribute name="CLASS" value="CAPACITOR"/>
-<attribute name="DESCRIPTION" value="CAP TANT 100UF 10%% 6.3V 2312"/>
+<attribute name="DESCRIPTION" value="CAP TANT 100UF 10% 6.3V 2312"/>
 <attribute name="LINK" value="https://www.digikey.de/product-detail/de/avx-corporation/TPSC107K006R0150/478-1764-1-ND"/>
 <attribute name="MANUFACTURER" value="AVX Corporation"/>

Commit message: sfp-breakout: increase pad size for DC barrel conn
... as done for all recent projects for Kaempfe (by updating from the
resp. Wuerth lib)
Parts:
- C1, C3, C9: DATASHEET (none) -> https://www.samsungsem.com/kr/support/product-search/mlcc/C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; DESCRIPTION CAP CER 10UF 16V X5R 0805 -> CAP CER 10UF 16V X5R 1206; LINK https://www.digikey.de/product-detail/de/samsung-electro-me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 -> https://www.digikey.com/en/products/detail/samsung-electro-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; MANUFACTURERPARTNUMBER CL21A106KOCLRNC -> CL31A106KOHNNNE; ROHSCERTIFICATE Bleifrei / RoHS-konform -> ROHS3 Compliant; SOURCEPARTNUMBER 1276-2399-1-ND -> 1276-1137-1-ND
- C2, C4, C5, C7, C8: DATASHEET (none) -> http://www.samsungsem.com/kr/support/product-search/mlcc/CL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; LINK http://www.digikey.de/product-detail/de/foo/1276-1005-1-ND -> https://www.digikey.com/product-detail/en/samsung-electro-m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; ROHSCERTIFICATE Bleifrei / RoHS-konform -> ROHS3 Compliant
- C6: DATASHEET (none) -> https://datasheets.avx.com/TPS.pdf; LINK https://www.digikey.de/product-detail/de/avx-corporation/TP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 -> https://www.digikey.com/product-detail/en/avx-corporation/T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; ROHSCERTIFICATE Bleifrei / RoHS-konform -> ROHS3 Compliant
- D1: DATASHEET (none) -> https://www.diodes.com/assets/Datasheets/B220_A-B260_A.pdf; DESCRIPTION DIODE SCHOTTKY 60V 1A SMA -> DIODE SCHOTTKY 60V 2A SMA; LINK https://www.digikey.de/product-detail/de/on-semiconductor/M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 -> https://www.digikey.com/en/products/detail/diodes-incorpora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; MANUFACTURER ON Semiconductor -> Diodes Incorporated; MANUFACTURERPARTNUMBER MBRA160T3G -> B260A-13-F; ROHSCERTIFICATE RoHS3-konform -> ROHS3 Compliant; SOURCEPARTNUMBER MBRA160T3GOSCT-ND -> B260A-FDICT-ND
- D2: DATASHEET (none) -> https://www.we-online.de/katalog/datasheet/824500500.pdf; LINK https://www.digikey.de/product-detail/de/wurth-electronics-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 -> https://www.digikey.com/product-detail/en/w-rth-elektronik/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; MANUFACTURER Wurth Electronics Inc. -> Würth Elektronik; ROHSCERTIFICATE Bleifrei / RoHS-konform -> ROHS3 Compliant
- J1: device sfp-breakout:694108106102 -> Wurth_Elektronik_Electromechanic_DC_Power_Jack_Connectors_rev15c:694108106102; DATASHEET (none) -> https://www.cuidevices.com/product/resource/pj-002bh-smt-tr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; LINK https://www.digikey.de/product-detail/de/cui-inc/PJ-002BH-S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 -> https://www.digikey.com/product-detail/en/cui-devices/PJ-00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; ROHSCERTIFICATE RoHS-konform -> RoHS Compliant
- L1, L2: DATASHEET (none) -> https://abracon.com/Magnetics/new/AIMC-0603.pdf; LINK https://www.digikey.de/product-detail/de/abracon-llc/AIMC-0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 -> https://www.digikey.com/product-detail/en/abracon-llc/AIMC-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; ROHSCERTIFICATE RoHS-konform -> RoHS Compliant
- R1, R2, R3, R4, R5, R7, R8: DATASHEET (none) -> https://www.seielect.com/catalog/sei-rmcf_rmcp.pdf; DESCRIPTION RES 10K OHM 1%% 1/10W 0603 -> RES 10K OHM 1% 1/10W 0603; LINK https://www.digikey.de/product-detail/de/stackpole-electron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 -> https://www.digikey.com/product-detail/en/stackpole-electro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; ROHSCERTIFICATE RoHS3-konform -> ROHS3 Compliant
- R10, R9: DATASHEET (none) -> https://www.yageo.com/upload/media/product/productsearch/da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; DESCRIPTION RES SMD 330 OHM 1%% 1/10W 0603 -> RES SMD 330 OHM 1% 1/10W 0603; LINK https://www.digikey.de/product-detail/de/yageo/RC0603FR-073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 -> https://www.digikey.com/product-detail/en/yageo/RC0603FR-07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; ROHSCERTIFICATE RoHS3-konform -> ROHS3 Compliant
- SFP1: DATASHEET (none) -> https://media.digikey.com/pdf/Data%20Sheets/Amphenol%20PDFs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; LINK https://www.digikey.de/product-detail/de/amphenol-icc-comme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 -> https://www.digikey.com/product-detail/en/amphenol-icc-comm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; ROHSCERTIFICATE Bleifrei / RoHS-konform -> RoHS Compliant
- T1, T2: DATASHEET (none) -> https://assets.nexperia.com/documents/data-sheet/BC847_SER.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; LINK https://www.digikey.de/product-detail/de/nexperia-usa-inc/B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 -> https://www.digikey.com/product-detail/en/nexperia-usa-inc/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; ROHSCERTIFICATE RoHS3-konform -> ROHS3 Compliant
- U1: DATASHEET (none) -> https://ww1.microchip.com/downloads/en/DeviceDoc/22056b.pdf; LINK https://www.digikey.de/product-detail/de/microchip-technolo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 -> https://www.digikey.com/en/products/detail/microchip-techno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; ROHSCERTIFICATE Bleifrei / RoHS-konform -> ROHS3 Compliant
