File: pico-pcm-cardem/pico-pcm-cardem.sch (EAGLE design)
At the start: 22 parts, among them IC1 MIC2091-1, U1 TXU0304BQA, U2 RASPBERRY_PICOSMD-TH, X1 FCI_FPC_REBEL_SFW6R-1, X2 JACK2.5_SJ-2523, X3 JACK2.5_SJ-2523

Commit message: pico-pcm-cardem: add various bom annotations
Parts:
- C1, C2, C3, C4: CLASS (none) -> CAPACITOR; DESCRIPTION (none) -> NO DESCRIPTION; LINK (none) -> UNKNOWN LINK; MANUFACTURER (none) -> UNKNOWN MANUFACTURER; MANUFACTURERPARTNUMBER (none) -> UNKNOWN MANUFACTURER PART NUMBER; POPULATED (none) -> TRUE; ROHSCERTIFICATE (none) -> UNKNOWN ROHS CERTIFICATE; SOURCE (none) -> UNKNOWN SOURCE; SOURCEPARTNUMBER (none) -> UNKNOWN SOURCE PART NUMBER
- IC1: CLASS (none) -> UNKNOWN CLASS; DESCRIPTION (none) -> NO DESCRIPTION; LINK (none) -> https://www.digikey.de/en/products/detail/microchip-technol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; MANUFACTURER (none) -> UNKNOWN MANUFACTURER; MANUFACTURERPARTNUMBER (none) -> https://www.digikey.de/en/products/detail/microchip-technol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; POPULATED (none) -> TRUE; ROHSCERTIFICATE (none) -> UNKNOWN ROHS CERTIFICATE; SOURCE (none) -> UNKNOWN SOURCE; SOURCEPARTNUMBER (none) -> 576-3891-1-ND
- JP1, JP2, JP3: CLASS (none) -> CONNECTOR\JUMPER; DESCRIPTION (none) -> NO DESCRIPTION; LINK (none) -> UNKNOWN LINK; MANUFACTURER (none) -> UNKNOWN MANUFACTURER; MANUFACTURERPARTNUMBER (none) -> UNKNOWN MANUFACTURER PART NUMBER; POPULATED (none) -> TRUE; ROHSCERTIFICATE (none) -> UNKNOWN ROHS CERTIFICATE; SOURCE (none) -> UNKNOWN SOURCE; SOURCEPARTNUMBER (none) -> UNKNOWN SOURCE PART NUMBER
- LED1: CLASS (none) -> LED; DESCRIPTION (none) -> NO DESCRIPTION; LINK (none) -> UNKNOWN LINK; MANUFACTURER (none) -> UNKNOWN MANUFACTURER; MANUFACTURERPARTNUMBER (none) -> UNKNOWN MANUFACTURER PART NUMBER; POPULATED (none) -> TRUE; ROHSCERTIFICATE (none) -> UNKNOWN ROHS CERTIFICATE; SOURCE (none) -> UNKNOWN SOURCE; SOURCEPARTNUMBER (none) -> UNKNOWN SOURCE PART NUMBER
- R1, R2, R3, R4, R5, R6, R7: CLASS (none) -> RESISTOR; DESCRIPTION (none) -> NO DESCRIPTION; LINK (none) -> UNKNOWN LINK; MANUFACTURER (none) -> UNKNOWN MANUFACTURER; MANUFACTURERPARTNUMBER (none) -> UNKNOWN MANUFACTURER PART NUMBER; POPULATED (none) -> TRUE; ROHSCERTIFICATE (none) -> UNKNOWN ROHS CERTIFICATE; SOURCE (none) -> UNKNOWN SOURCE; SOURCEPARTNUMBER (none) -> UNKNOWN SOURCE PART NUMBER
- SIM1: CLASS (none) -> UNKNOWN CLASS; DESCRIPTION (none) -> NO DESCRIPTION; LINK (none) -> UNKNOWN LINK; MANUFACTURER (none) -> UNKNOWN MANUFACTURER; MANUFACTURERPARTNUMBER (none) -> UNKNOWN MANUFACTURER PART NUMBER; POPULATED (none) -> TRUE; ROHSCERTIFICATE (none) -> UNKNOWN ROHS CERTIFICATE; SOURCE (none) -> UNKNOWN SOURCE; SOURCEPARTNUMBER (none) -> UNKNOWN SOURCE PART NUMBER
- U1: CLASS (none) -> IC; DESCRIPTION (none) -> NO DESCRIPTION; LINK (none) -> https://www.digikey.de/en/products/detail/texas-instruments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; MANUFACTURER (none) -> UNKNOWN MANUFACTURER; MANUFACTURERPARTNUMBER (none) -> TXU0304BQAR; POPULATED (none) -> TRUE; ROHSCERTIFICATE (none) -> UNKNOWN ROHS CERTIFICATE; SOURCE (none) -> UNKNOWN SOURCE; SOURCEPARTNUMBER (none) -> 296-TXU0304BQARCT-ND
- U2: CLASS (none) -> IC; DESCRIPTION (none) -> NO DESCRIPTION; LINK (none) -> https://www.digikey.de/en/products/detail/raspberry-pi/SC09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; MANUFACTURER (none) -> UNKNOWN MANUFACTURER; MANUFACTURERPARTNUMBER (none) -> UNKNOWN MANUFACTURER PART NUMBER; POPULATED (none) -> TRUE; ROHSCERTIFICATE (none) -> UNKNOWN ROHS CERTIFICATE; SOURCE (none) -> UNKNOWN SOURCE; SOURCEPARTNUMBER (none) -> 2648-SC0915CT-ND
- X1: CLASS (none) -> CONNECTOR; DESCRIPTION (none) -> NO DESCRIPTION; LINK (none) -> https://www.digikey.de/en/products/detail/amphenol-cs-fci/S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; MANUFACTURER (none) -> UNKNOWN MANUFACTURER; MANUFACTURERPARTNUMBER (none) -> SFW6R-1STE1LF; POPULATED (none) -> TRUE; ROHSCERTIFICATE (none) -> UNKNOWN ROHS CERTIFICATE; SOURCE (none) -> UNKNOWN SOURCE; SOURCEPARTNUMBER (none) -> 609-1889-1-ND
- X2: CLASS (none) -> CONNECTOR; DESCRIPTION (none) -> NO DESCRIPTION; LINK (none) -> UNKNOWN LINK; MANUFACTURER (none) -> UNKNOWN MANUFACTURER; MANUFACTURERPARTNUMBER (none) -> UNKNOWN MANUFACTURER PART NUMBER; POPULATED (none) -> TRUE; ROHSCERTIFICATE (none) -> UNKNOWN ROHS CERTIFICATE; SOURCE (none) -> UNKNOWN SOURCE; SOURCEPARTNUMBER (none) -> UNKNOWN SOURCE PART NUMBER
- X3: CLASS (none) -> CONNECTOR; DESCRIPTION (none) -> NO DESCRIPTION; LINK (none) -> https://www.digikey.de/en/products/detail/cui-devices/SJ-25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; MANUFACTURER (none) -> UNKNOWN MANUFACTURER; MANUFACTURERPARTNUMBER (none) -> SJ-2523-SMT-TR; POPULATED (none) -> TRUE; ROHSCERTIFICATE (none) -> UNKNOWN ROHS CERTIFICATE; SOURCE (none) -> UNKNOWN SOURCE; SOURCEPARTNUMBER (none) -> CP-2523SJCT-ND
